Commit message: minor updates

File: skidy_description/urdf/robot_test_diff_drive.urdf (robot description, URDF)
Before this commit: robot device, 5 links, 4 joints
Links:
- link imu_link: geometry collision box size=0.01 0.01 0.01; visual box size=0.01 0.01 0.01
- link navsat_link: geometry collision box size=0.01 0.01 0.01; visual box size=0.01 0.01 0.01
Joints:
- joint imu_joint: origin xyz=0 0 0.01 -> xyz=0.0 ${base_width/2} ${base_height/2+0.01}
- joint navsat_joint: origin xyz=-0.2 0.3 0.3 rpy=0 0 0 -> xyz=0.0 -${base_width/2} ${base_height/2+0.01}

File: skidy_description/urdf/sensors/camera.gazebo.xacro (robot description, xacro)
@@ -1,10 +1,31 @@
 <?xml version="1.0"?>
 <robot xmlns:xacro="http://ros.org/wiki/xacro">
-    <xacro:macro name="depth_camera_sensor" params="reference_link sensor_name update_rate topic_ns topic">
+    <xacro:include filename="$(find skidy_description)/urdf/robot_diff_drive.xacro" />
+    <xacro:macro name="depth_camera_sensor" params="reference_link parent sensor_name update_rate topic_ns topic">
+        <link name="${reference_link}">
+            <visual>
+                <geometry>
+                    <box size="0.05 0.05 0.05"/>
+                </geometry>
+            </visual>
+            <collision>
+                <geometry>
+                    <box size="0.05 0.05 0.05"/>
+                </geometry>
+            </collision>
+            <xacro:box_inertia m="0.01" w="0.01" d="0.01" h="0.01"/>
+        </link>
+        <joint name="camera_joint" type="fixed">
+            <parent link="${parent}"/>
+            <child link="${reference_link}"/>
+            <origin xyz="0 0 0.58" rpy="0 0 0"/>
+        </joint>
         <gazebo reference="${reference_link}">
                 <always_on>1</always_on>
-                <sensor name="${sensor_name}" type="depth_camera">
+                <sensor name="${sensor_name}" type="rgbd_camera">
                     <update_rate>${update_rate}</update_rate>
                     <topic>${topic_ns}/${topic}</topic>
+                    <ignition_frame_id>"camera_link"</ignition_frame_id>
+                    <always_on>1</always_on>
                     <camera>
                         <horizontal_fov>1.05</horizontal_fov>

File: skidy_description/urdf/sensors/d435.gazebo.xacro (robot description, xacro)
@@ -32,6 +32,6 @@
         <joint name="${name}_joint" type="fixed">
 <!--            <xacro:insert_block name="origin" />-->
-<!--            <origin xyz="-0.5 0 0.8" rpy="-1.7450 0 -1.57"/>&ndash;&gt;-->
-            <origin xyz="0 0 0.18" rpy="0 0.05 0"/>-->
+<!--            <origin xyz="-0.5 0 0.8" rpy="-1.7450 0 -1.57"/>-->
+            <origin xyz="0 0 0.18" rpy="0 0.05 0"/>
             <parent link="${parent}"/>
             <child link="${name}_bottom_screw_frame" />
@@ -137,6 +137,6 @@
                 <!--            this is detected by ros2 run tf2_ros tf2_echo camera_bottom_screw_frame camera_depth_optical_frame-->
                 <!--                <pose>0.0 0.020 0.011 0.0 0.0 0.0</pose>-->
+                <ignition_frame_id>"${name}_color_optical_frame"</ignition_frame_id>
                 <camera>
-<!--                    <optical_frame_id>"${name}_color_optical_frame"</optical_frame_id>-->
                     <horizontal_fov>1.047</horizontal_fov>
                     <image>
