Commit message: updates

File: skidy_description/urdf/sensors/d435.gazebo.xacro (robot description, xacro)
@@ -33,5 +33,5 @@
 <!--            <xacro:insert_block name="origin" />-->
 <!--            <origin xyz="-0.5 0 0.8" rpy="-1.7450 0 -1.57"/>&ndash;&gt;-->
-            <origin xyz="0 0 0.28" rpy="0 0.05 0"/>-->
+            <origin xyz="0 0 0.18" rpy="0 0.05 0"/>-->
             <parent link="${parent}"/>
             <child link="${name}_bottom_screw_frame" />

File: skidy_description/urdf/sensors/navsat.gazebo.xacro (robot description, xacro)
@@ -13,5 +13,5 @@
             <sensor name="navsat" type="navsat">
                 <always_on>1</always_on>
-                <update_rate>1</update_rate>
+                <update_rate>${update_rate}</update_rate>
                 <pose>0 0 0.05 0 0 0</pose>
                 <topic>${topic_ns}/${topic}</topic>
